Commit message: working urdf w

File: anthropmass/anthropmass/mass/model_output/simple_human.urdf (robot description, URDF)
Before this commit: robot simple_human, 17 links, 16 joints
Joints:
- joint forearm_to_hand: origin xyz=0 0 -0.09064928442239761 rpy=0 0 0 -> xyz=0 0 -0.09796416759490967 rpy=0 0 0
- joint forearm_to_hand_right: origin xyz=0 0 -0.09064928442239761 rpy=0 0 0 -> xyz=0 0 -0.09796416759490967 rpy=0 0 0
- joint lower_leg_left_to_foot: origin xyz=0.08745751157402992 0 -0.06745107471942902 rpy=0 0 1.57 -> xyz=0.10210202634334564 0 -0.07403331995010376 rpy=0 0 1.57
- joint lower_leg_right_to_foot: origin xyz=0.08745751157402992 0 -0.06745107471942902 rpy=0 0 1.57 -> xyz=0.10210202634334564 0 -0.07403331995010376 rpy=0 0 1.57
- joint torso_bottom_to_mid: origin xyz=0 0 0.14929187297821045 rpy=0 0 0 -> xyz=0 0 0.16574005782604218 rpy=0 0 0
- joint torso_bottom_to_upper_leg_left: origin xyz=0 -0.06983193755149841 -0.35980966687202454 rpy=0 0 0 -> xyz=0 -0.07464926689863205 -0.4176444113254547 rpy=0 0 0
- joint torso_bottom_to_upper_leg_right: origin xyz=0 0.06983193755149841 -0.35980966687202454 rpy=0 0 0 -> xyz=0 0.07464926689863205 -0.4176444113254547 rpy=0 0 0
- joint torso_mid_to_top: origin xyz=0 0 0.22390228509902954 rpy=0 0 0 -> xyz=0 0 0.22864733636379242 rpy=0 0 0
- joint torso_mid_to_upper_arm_left: origin xyz=0 -0.290840320289135 0.035485073924064636 rpy=0 0 1.57 -> xyz=0 -0.2639159820973873 0.010754510760307312 rpy=0 0 1.57
- joint torso_mid_to_upper_arm_right: origin xyz=0 0.290840320289135 0.035485073924064636 rpy=0 0 -1.57 -> xyz=0 0.2639159820973873 0.010754510760307312 rpy=0 0 -1.57
- joint torso_top_to_neck: origin xyz=0 0 0.2077152170240879 rpy=0 0 0 -> xyz=0 0 0.24094677716493607 rpy=0 0 0
- joint upper_arm_left_to_forearm: origin xyz=0 0 -0.2657824754714966 rpy=0 0 0 -> xyz=0 0 -0.2944090664386749 rpy=0 0 0
- joint upper_arm_right_to_forearm: origin xyz=0 0 -0.2657824754714966 rpy=0 0 0 -> xyz=0 0 -0.2944090664386749 rpy=0 0 0
- joint upper_leg_left_to_lower_leg: origin xyz=0 0 -0.3706740140914917 rpy=0 0 0 -> xyz=0 0 -0.43394097685813904 rpy=0 0 0
- joint upper_leg_right_to_lower_leg: origin xyz=0 0 -0.3706740140914917 rpy=0 0 0 -> xyz=0 0 -0.43394097685813904 rpy=0 0 0

Commit message: Big Update BSP

File: anthropmass/anthropmass/mass/model_output/simple_human.urdf (robot description, URDF)
Before this commit: robot simple_human, 17 links, 16 joints
Joints:
- joint forearm_to_hand: axis 0 0 0 -> 0 0 1; limit (none) -> lower=-1.57 upper=1.57 effort=1 velocity=1; origin xyz=0 0 -0.09796416759490967 rpy=0 0 0 -> xyz=0.000000 0.000000 -0.153549 rpy=0 0 1.57; type fixed -> revolute
- joint forearm_to_hand_right: axis 0 0 0 -> 0 0 1; limit (none) -> lower=-1.57 upper=1.57 effort=1 velocity=1; origin xyz=0 0 -0.09796416759490967 rpy=0 0 0 -> xyz=0.000000 0.000000 -0.153549 rpy=0 0 1.57; type fixed -> revolute
- joint lower_leg_left_to_foot: axis 0 0 0 -> 0 0 1; limit (none) -> lower=-1.57 upper=1.57 effort=1 velocity=1; origin xyz=0.10210202634334564 0 -0.07403331995010376 rpy=0 0 1.57 -> xyz=0.000000 -0.094517 -0.214511 rpy=0 0 -1.57; type fixed -> revolute
- joint lower_leg_right_to_foot: axis 0 0 0 -> 0 0 1; limit (none) -> lower=-1.57 upper=1.57 effort=1 velocity=1; origin xyz=0.10210202634334564 0 -0.07403331995010376 rpy=0 0 1.57 -> xyz=0.000000 -0.094517 -0.214511 rpy=0 0 1.57; type fixed -> revolute
- joint neck_to_head: axis 0 0 0 -> 0 0 1; limit (none) -> lower=-1.57 upper=1.57 effort=1 velocity=1; origin xyz=0 0 0 rpy=0 0 0 -> xyz=0.000000 0.000000 0.153979 rpy=0 0 0; type fixed -> revolute
- joint torso_bottom_to_mid: axis 0 0 0 -> 0 0 1; limit (none) -> lower=-1.57 upper=1.57 effort=1 velocity=1; origin xyz=0 0 0.16574005782604218 rpy=0 0 0 -> xyz=0.000000 0.000000 0.165613 rpy=0 0 0; type fixed -> revolute
- joint torso_bottom_to_upper_leg_left: axis 0 0 0 -> 0 0 1; limit (none) -> lower=-1.57 upper=1.57 effort=1 velocity=1; origin xyz=0 -0.07464926689863205 -0.4176444113254547 rpy=0 0 0 -> xyz=0.080021 0.000000 -0.274166 rpy=0 0 0; type fixed -> revolute
- joint torso_bottom_to_upper_leg_right: axis 0 0 0 -> 0 0 1; limit (none) -> lower=-1.57 upper=1.57 effort=1 velocity=1; origin xyz=0 0.07464926689863205 -0.4176444113254547 rpy=0 0 0 -> xyz=-0.080021 0.000000 -0.274166 rpy=0 0 0; type fixed -> revolute
- joint torso_mid_to_top: axis 0 0 0 -> 0 0 1; limit (none) -> lower=-1.57 upper=1.57 effort=1 velocity=1; origin xyz=0 0 0.22864733636379242 rpy=0 0 0 -> xyz=0.000000 0.000000 0.176500 rpy=0 0 0; type fixed -> revolute
- joint torso_mid_to_upper_arm_left: axis 0 0 0 -> 0 0 1; limit (none) -> lower=-1.57 upper=1.57 effort=1 velocity=1; origin xyz=0 -0.2639159820973873 0.010754510760307312 rpy=0 0 1.57 -> xyz=0.173491 0.000000 0.094494 rpy=0 0 1.57; type fixed -> revolute
- joint torso_mid_to_upper_arm_right: axis 0 0 0 -> 0 0 1; limit (none) -> lower=-1.57 upper=1.57 effort=1 velocity=1; origin xyz=0 0.2639159820973873 0.010754510760307312 rpy=0 0 -1.57 -> xyz=-0.173491 0.000000 0.094494 rpy=0 0 -1.57; type fixed -> revolute
- joint torso_top_to_neck: axis 0 0 0 -> 0 0 1; limit (none) -> lower=-1.57 upper=1.57 effort=1 velocity=1; origin xyz=0 0 0.24094677716493607 rpy=0 0 0 -> xyz=0.000000 0.000000 0.119967 rpy=0 0 0; type fixed -> revolute
- joint upper_arm_left_to_forearm: axis 0 0 1 -> 1 0 0; origin xyz=0 0 -0.2944090664386749 rpy=0 0 0 -> xyz=0.000000 0.000000 -0.292638 rpy=0 0 0
- joint upper_arm_right_to_forearm: origin xyz=0 0 -0.2944090664386749 rpy=0 0 0 -> xyz=0.000000 0.000000 -0.292638 rpy=0 0 0
- joint upper_leg_left_to_lower_leg: origin xyz=0 0 -0.43394097685813904 rpy=0 0 0 -> xyz=0.000000 0.000000 -0.418467 rpy=0 0 0
- joint upper_leg_right_to_lower_leg: origin xyz=0 0 -0.43394097685813904 rpy=0 0 0 -> xyz=0.000000 0.000000 -0.418467 rpy=0 0 0

Commit message: 1000 fix

File: anthropmass/anthropmass/mass/model_output/simple_human.urdf (robot description, URDF)
Before this commit: robot simple_human, 17 links, 16 joints
Joints:
- joint forearm_to_hand: origin xyz=0.000000 0.000000 -0.153549 rpy=0 0 1.57 -> xyz=0.000000 0.000000 -0.166337 rpy=0 0 1.57
- joint forearm_to_hand_right: origin xyz=0.000000 0.000000 -0.153549 rpy=0 0 1.57 -> xyz=0.000000 0.000000 -0.166337 rpy=0 0 1.57
- joint lower_leg_left_to_foot: origin xyz=0.000000 -0.094517 -0.214511 rpy=0 0 -1.57 -> xyz=0.000000 -0.107559 -0.235179 rpy=0 0 -1.57
- joint lower_leg_right_to_foot: origin xyz=0.000000 -0.094517 -0.214511 rpy=0 0 1.57 -> xyz=0.000000 -0.107559 -0.235179 rpy=0 0 1.57
- joint neck_to_head: origin xyz=0.000000 0.000000 0.153979 rpy=0 0 0 -> xyz=0.000000 0.000000 0.157872 rpy=0 0 0
- joint torso_bottom_to_mid: origin xyz=0.000000 0.000000 0.165613 rpy=0 0 0 -> xyz=0.000000 0.000000 0.202507 rpy=0 0 0
- joint torso_bottom_to_upper_leg_left: origin xyz=0.080021 0.000000 -0.274166 rpy=0 0 0 -> xyz=0.081762 0.000000 -0.306132 rpy=0 0 0
- joint torso_bottom_to_upper_leg_right: origin xyz=-0.080021 0.000000 -0.274166 rpy=0 0 0 -> xyz=-0.081762 0.000000 -0.306132 rpy=0 0 0
- joint torso_mid_to_top: origin xyz=0.000000 0.000000 0.176500 rpy=0 0 0 -> xyz=0.000000 0.000000 0.211951 rpy=0 0 0
- joint torso_mid_to_upper_arm_left: origin xyz=0.173491 0.000000 0.094494 rpy=0 0 1.57 -> xyz=0.171764 0.000000 0.127444 rpy=0 0 1.57
- joint torso_mid_to_upper_arm_right: origin xyz=-0.173491 0.000000 0.094494 rpy=0 0 -1.57 -> xyz=-0.171764 0.000000 0.127444 rpy=0 0 -1.57
- joint torso_top_to_neck: origin xyz=0.000000 0.000000 0.119967 rpy=0 0 0 -> xyz=0.000000 0.000000 0.130991 rpy=0 0 0
- joint upper_arm_left_to_forearm: origin xyz=0.000000 0.000000 -0.292638 rpy=0 0 0 -> xyz=0.000000 0.000000 -0.314382 rpy=0 0 0
- joint upper_arm_right_to_forearm: origin xyz=0.000000 0.000000 -0.292638 rpy=0 0 0 -> xyz=0.000000 0.000000 -0.314382 rpy=0 0 0
- joint upper_leg_left_to_lower_leg: origin xyz=0.000000 0.000000 -0.418467 rpy=0 0 0 -> xyz=0.000000 0.000000 -0.461928 rpy=0 0 0
- joint upper_leg_right_to_lower_leg: origin xyz=0.000000 0.000000 -0.418467 rpy=0 0 0 -> xyz=0.000000 0.000000 -0.461928 rpy=0 0 0

Commit message: upade final result comments

File: anthropmass/anthropmass/mass/model_output/simple_human.urdf (robot description, URDF)
Before this commit: robot simple_human, 17 links, 16 joints
Joints:
- joint forearm_to_hand: origin xyz=0.000000 0.000000 -0.166337 rpy=0 0 1.57 -> xyz=0.000000 0.000000 -0.158372 rpy=0 0 1.57
- joint forearm_to_hand_right: origin xyz=0.000000 0.000000 -0.166337 rpy=0 0 1.57 -> xyz=0.000000 0.000000 -0.158372 rpy=0 0 1.57
- joint lower_leg_left_to_foot: origin xyz=0.000000 -0.107559 -0.235179 rpy=0 0 -1.57 -> xyz=0.000000 -0.099630 -0.208102 rpy=0 0 -1.57
- joint lower_leg_right_to_foot: origin xyz=0.000000 -0.107559 -0.235179 rpy=0 0 1.57 -> xyz=0.000000 -0.099630 -0.208102 rpy=0 0 1.57
- joint neck_to_head: origin xyz=0.000000 0.000000 0.157872 rpy=0 0 0 -> xyz=0.000000 0.000000 0.163569 rpy=0 0 0
- joint torso_bottom_to_mid: origin xyz=0.000000 0.000000 0.202507 rpy=0 0 0 -> xyz=0.000000 0.000000 0.196715 rpy=0 0 0
- joint torso_bottom_to_upper_leg_left: origin xyz=0.081762 0.000000 -0.306132 rpy=0 0 0 -> xyz=0.073802 0.000000 -0.283862 rpy=0 0 0
- joint torso_bottom_to_upper_leg_right: origin xyz=-0.081762 0.000000 -0.306132 rpy=0 0 0 -> xyz=-0.073802 0.000000 -0.283862 rpy=0 0 0
- joint torso_mid_to_top: origin xyz=0.000000 0.000000 0.211951 rpy=0 0 0 -> xyz=0.000000 0.000000 0.192782 rpy=0 0 0
- joint torso_mid_to_upper_arm_left: origin xyz=0.171764 0.000000 0.127444 rpy=0 0 1.57 -> xyz=0.188175 0.000000 0.100139 rpy=0 0 1.57
- joint torso_mid_to_upper_arm_right: origin xyz=-0.171764 0.000000 0.127444 rpy=0 0 -1.57 -> xyz=-0.188175 0.000000 0.100139 rpy=0 0 -1.57
- joint torso_top_to_neck: origin xyz=0.000000 0.000000 0.130991 rpy=0 0 0 -> xyz=0.000000 0.000000 0.115913 rpy=0 0 0
- joint upper_arm_left_to_forearm: origin xyz=0.000000 0.000000 -0.314382 rpy=0 0 0 -> xyz=0.000000 0.000000 -0.301917 rpy=0 0 0
- joint upper_arm_right_to_forearm: origin xyz=0.000000 0.000000 -0.314382 rpy=0 0 0 -> xyz=0.000000 0.000000 -0.301917 rpy=0 0 0
- joint upper_leg_left_to_lower_leg: origin xyz=0.000000 0.000000 -0.461928 rpy=0 0 0 -> xyz=0.000000 0.000000 -0.412969 rpy=0 0 0
- joint upper_leg_right_to_lower_leg: origin xyz=0.000000 0.000000 -0.461928 rpy=0 0 0 -> xyz=0.000000 0.000000 -0.412969 rpy=0 0 0
